File: ardFilaSplice/KiCad/ardFilaSplice/ardFilaSplice.sch (KiCad schematic (older format))
At the start: 18 parts, among them J1 2-pin_fan_output_header, J2 3-pin_KY-019_relay_header, K1 SANYOU_SRD_Form_C, Q1 20N6003, U1 KY-040_Rotary_Encoder, U2 2-pole_power_in_screw_terminal, U3 Arduino_Mini_Pro, U4 TM1637_4x7-segment_display, U5 L7805, U6 4-pole_Heater_thermistor_scre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

Commit message: ardFilaSplice sketch
Parts:
- added R3: 10k, My_Misc:R_Axial_DIN0207_L6.3mm_D2.5mm_P10.16mm_Horizontal_larger_pads, symbol Device:R
Connections:
- net GND: now also R3.2
- net at Q1.1 (G), U3.9 (6): now also R3.1
Changed lines of the file:
@@
 L power:GND #PWR08
 U 1 1 5FF645A2
-P 5000 7150
-F 0 "#PWR08" H 5000 6900 50  0001 C CNN
-F 1 "GND" H 5005 6977 50  0000 C CNN
-F 2 "" H 5000 7150 50  0001 C CNN
-F 3 "" H 5000 7150 50  0001 C CNN
-	1    5000 7150
+P 5000 7450
+F 0 "#PWR08" H 5000 7200 50  0001 C CNN
+F 1 "GND" H 5005 7277 50  0000 C CNN
+F 2 "" H 5000 7450 50  0001 C CNN
+F 3 "" H 5000 7450 50  0001 C CNN
+	1    5000 7450
 	1    0    0    -1
 $EndComp
 Wire Wire Line
-	5000 7050 5000 7150
+	5000 7050 5000 7400
 Wire Wire Line
 	4700 6850 4350 6850
@@
 Wire Wire Line
 	1800 2450 1800 2550
+$Comp
+L Device:R R3
+U 1 1 5FE8B6A2
+P 4350 7150
+F 0 "R3" H 4420 7196 50  0000 L CNN
+F 1 "10k" H 4420 7105 50  0000 L CNN
+F 2 "My_Misc:R_Axial_DIN0207_L6.3mm_D2.5mm_P10.16mm_Horizontal_larger_pads" V 4280 7150 50  0001 C CNN
+F 3 "~" H 4350 7150 50  0001 C CNN
+	1    4350 7150
+	1    0    0    -1
+$EndComp
+Wire Wire Line
+	4350 6850 4350 7000
+Connection ~ 4350 6850
+Wire Wire Line
+	4350 7300 4350 7400
+Wire Wire Line
+	4350 7400 5000 7400
+Connection ~ 5000 7400
+Wire Wire Line
+	5000 7400 5000 7450
 $EndSCHEMATC
