File: ardUnoTester/LEDs.kicad_sch (KiCad schematic)
At the start: 42 parts

Commit message: page settings
Other:
- title: (none) -> ardUnoTester
Changed lines of the file:
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@@
 (kicad_sch (version 20211123) (generator eeschema)
   (paper "A4")
+  (title_block
+    (title "ardUnoTester")
+    (date "2022-09-18")
+    (rev "0.1")
+  )
   (wire (pts (xy 86.36 66.04) (xy 91.44 66.04))
     (stroke (width 0) (type default) (color 0 0 0 0))
