File: ardUnoTester/ardUnoTester.kicad_pcb (KiCad board)
At the start: 2 copper layers, 122 x 110 mm, 48 parts, among them U1 Power In

Commit message: page settings
Other:
- board text added: "${TITLE}-${REVISION} Design: Jon Sagebrand github.com/jonsag/miscArduino"
Changed lines of the file:
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@@
   )
   (paper "A4")
+  (title_block
+    (title "ardUnoTester")
+    (date "2022-09-18")
+    (rev "0.1")
+  )
   (layers
     (0 "F.Cu" signal)
@@
   (gr_line (start 46.8 146) (end 46.8 36) (layer "Edge.Cuts") (width 0.1))
   (gr_line (start 168.8 146) (end 46.8 146) (layer "Edge.Cuts") (width 0.1))
+  (gr_text "${TITLE}-${REVISION}\nDesign: Jon Sagebrand\ngithub.com/jonsag/miscArduino" (at 165 124) (layer "B.Cu")
+    (effects (font (size 2.286 2.286) (thickness 0.381)) (justify left mirror))
+  )
   (segment (start 71.21 134.2) (end 67.4 134.2) (width 0.762) (layer "B.Cu") (net 1))
   (segment (start 71.295 127) (end 67.485 127) (width 0.762) (layer "B.Cu") (net 2))
