File: ardUnoTester/ardUnoTester.kicad_sch (KiCad schematic)
At the start: 6 parts, among them U1 Power In

Commit message: page settings
Other:
- title: (none) -> ardUnoTester
Changed lines of the file:
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@@
 (kicad_sch (version 20211123) (generator eeschema)
   (paper "A4")
+  (title_block
+    (title "ardUnoTester")
+    (date "2022-09-18")
+    (rev "0.1")
+  )
   (junction (at 142.24 120.65) (diameter 0) (color 0 0 0 0)
   )
