File: ATmega328-test-rig/ATmega328.kicad_sch (KiCad schematic)
At the start: 12 parts, among them J1 Power in, J2 FTDI, U1 AMS1117-5.0, U2 ATmega328P-PU, Y1 16MHz

Commit message: test rig
Parts:
- U2: footprint My_Misc:DIP-28_W7.62mm_LongPads w socket -> My_Misc:ZIF_DIP_Socket-28_W6.9_W7.62_W7.62_W12.7_W13.5_w_dip_packet_large
- renumbered J1 to J2, J2 to J3, JP1 to JP2, R1 to R19
Changed lines of the file:
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@@
     (property "Reference" "U2" (id 0) (at 119.38 54.0893 0))
     (property "Value" "ATmega328P-PU" (id 1) (at 119.38 56.6293 0))
-    (property "Footprint" "My_Misc:DIP-28_W7.62mm_LongPads w socket" (id 2) (at 142.24 88.9 0)
+    (property "Footprint" "My_Misc:ZIF_DIP_Socket-28_W6.9_W7.62_W7.62_W12.7_W13.5_w_dip_packet_large" (id 2) (at 142.24 88.9 0)
       (effects (font (size 1.27 1.27) italic) hide)
     )
@@
   (symbol (lib_id "power:VCC") (at 50.8 40.64 0) (unit 1)
     (in_bom yes) (on_board yes) (fields_autoplaced)
-    (property "Reference" "#PWR01" (id 0) (at 50.8 44.45 0)
+    (property "Reference" "#PWR04" (id 0) (at 50.8 44.45 0)
       (effects (font (size 1.27 1.27)) hide)
     )
@@
   (symbol (lib_id "My_Headers:6-pin_FTDI_header") (at 210.82 50.8 0) (unit 1)
     (in_bom yes) (on_board yes) (fields_autoplaced)
-    (property "Reference" "J2" (id 0) (at 211.455 40.64 0))
+    (property "Reference" "J3" (id 0) (at 211.455 40.64 0))
     (property "Value" "FTDI" (id 1) (at 211.455 43.18 0))
     (property "Footprint" "My_Headers:6-pin FTDI Programmer PinSocket large" (id 2) (at 210.82 50.8 0)
@@
   (symbol (lib_id "Device:R") (at 229.87 95.25 90) (unit 1)
     (in_bom yes) (on_board yes) (fields_autoplaced)
-    (property "Reference" "R1" (id 0) (at 229.87 88.9 90))
+    (property "Reference" "R19" (id 0) (at 229.87 88.9 90))
     (property "Value" "10k" (id 1) (at 229.87 91.44 90))
     (property "Footprint" "My_Misc:R_Axial_DIN0207_L6.3mm_D2.5mm_P10.16mm_Horizontal_larger_pads" (id 2) (at 229.87 97.028 90)
@@
   (symbol (lib_id "power:+5V") (at 226.06 26.67 0) (unit 1)
     (in_bom yes) (on_board yes) (fields_autoplaced)
-    (property "Reference" "#PWR011" (id 0) (at 226.06 30.48 0)
+    (property "Reference" "#PWR014" (id 0) (at 226.06 30.48 0)
       (effects (font (size 1.27 1.27)) hide)
     )
@@
   (symbol (lib_id "power:GND") (at 63.5 115.57 0) (unit 1)
     (in_bom yes) (on_board yes) (fields_autoplaced)
-    (property "Reference" "#PWR04" (id 0) (at 63.5 121.92 0)
+    (property "Reference" "#PWR07" (id 0) (at 63.5 121.92 0)
       (effects (font (size 1.27 1.27)) hide)
     )
@@
   (symbol (lib_id "power:VCC") (at 50.8 83.82 0) (unit 1)
     (in_bom yes) (on_board yes) (fields_autoplaced)
-    (property "Reference" "#PWR03" (id 0) (at 50.8 87.63 0)
+    (property "Reference" "#PWR06" (id 0) (at 50.8 87.63 0)
       (effects (font (size 1.27 1.27)) hide)
     )
@@
   (symbol (lib_id "power:GND") (at 50.8 54.61 0) (unit 1)
     (in_bom yes) (on_board yes) (fields_autoplaced)
-    (property "Reference" "#PWR02" (id 0) (at 50.8 60.96 0)
+    (property "Reference" "#PWR05" (id 0) (at 50.8 60.96 0)
       (effects (font (size 1.27 1.27)) hide)
     )
@@
   (symbol (lib_id "My_Headers:2-pin_power_input_header") (at 60.96 45.72 0) (unit 1)
     (in_bom yes) (on_board yes) (fields_autoplaced)
-    (property "Reference" "J1" (id 0) (at 62.23 46.9899 0)
+    (property "Reference" "J2" (id 0) (at 62.23 46.9899 0)
       (effects (font (size 1.27 1.27)) (justify left))
     )
@@
   (symbol (lib_id "power:+5V") (at 142.24 40.64 0) (unit 1)
     (in_bom yes) (on_board yes) (fields_autoplaced)
-    (property "Reference" "#PWR06" (id 0) (at 142.24 44.45 0)
+    (property "Reference" "#PWR09" (id 0) (at 142.24 44.45 0)
       (effects (font (size 1.27 1.27)) hide)
     )
@@
   (symbol (lib_id "power:+5V") (at 220.98 90.17 0) (unit 1)
     (in_bom yes) (on_board yes) (fields_autoplaced)
-    (property "Reference" "#PWR09" (id 0) (at 220.98 93.98 0)
+    (property "Reference" "#PWR012" (id 0) (at 220.98 93.98 0)
       (effects (font (size 1.27 1.27)) hide)
     )
@@
   (symbol (lib_id "power:+5V") (at 259.08 40.64 0) (unit 1)
     (in_bom yes) (on_board yes) (fields_autoplaced)
-    (property "Reference" "#PWR012" (id 0) (at 259.08 44.45 0)
+    (property "Reference" "#PWR015" (id 0) (at 259.08 44.45 0)
       (effects (font (size 1.27 1.27)) hide)
     )
@@
   (symbol (lib_id "power:GND") (at 220.98 139.7 0) (unit 1)
     (in_bom yes) (on_board yes) (fields_autoplaced)
-    (property "Reference" "#PWR010" (id 0) (at 220.98 146.05 0)
+    (property "Reference" "#PWR013" (id 0) (at 220.98 146.05 0)
       (effects (font (size 1.27 1.27)) hide)
     )
@@
   (symbol (lib_id "power:+5V") (at 76.2 83.82 0) (unit 1)
     (in_bom yes) (on_board yes) (fields_autoplaced)
-    (property "Reference" "#PWR05" (id 0) (at 76.2 87.63 0)
+    (property "Reference" "#PWR08" (id 0) (at 76.2 87.63 0)
       (effects (font (size 1.27 1.27)) hide)
     )
@@
   (symbol (lib_id "power:GND") (at 220.98 63.5 0) (unit 1)
     (in_bom yes) (on_board yes) (fields_autoplaced)
-    (property "Reference" "#PWR08" (id 0) (at 220.98 69.85 0)
+    (property "Reference" "#PWR011" (id 0) (at 220.98 69.85 0)
       (effects (font (size 1.27 1.27)) hide)
     )
@@
   (symbol (lib_id "power:GND") (at 142.24 137.16 0) (unit 1)
     (in_bom yes) (on_board yes) (fields_autoplaced)
-    (property "Reference" "#PWR07" (id 0) (at 142.24 143.51 0)
+    (property "Reference" "#PWR010" (id 0) (at 142.24 143.51 0)
       (effects (font (size 1.27 1.27)) hide)
     )
@@
   (symbol (lib_id "Jumper:Jumper_2_Open") (at 226.06 38.1 90) (unit 1)
     (in_bom yes) (on_board yes) (fields_autoplaced)
-    (property "Reference" "JP1" (id 0) (at 227.33 36.8299 90)
+    (property "Reference" "JP2" (id 0) (at 227.33 36.8299 90)
       (effects (font (size 1.27 1.27)) (justify right))
     )
