File: ATmega328base/ATmega328.kicad_sch (KiCad schematic)
At the start: 12 parts, among them J1 Power in, J2 FTDI, U1 AMS1117-5.0, U2 ATmega328P-PU, Y1 16MHz

Commit message: atmega328
Parts:
- added C3, C4: 100n, My_Misc:C_Disc_D4.3mm_W1.9mm_P5.00mm_large, symbol Device:C
- renumbered C3 to C5, C4 to C6, C5 to C7
Connections:
- net +5V: now also C3.1, C4.2
- net GND: now also C3.2, C4.1
- net AREF: now reaches U2.21 (AREF)
Other:
- moved on the sheet: U2
