File: ATmega328base-SMD/ATmega328base-SMD.kicad_pcb (KiCad board)
At the start: 2 copper layers, 11 parts, among them J1 FTDI, J2 Power in, U1 AMS1117-5_0, U2 ATMEGA328P-AU, X1 X322516MLB4SI

Commit message: atmega base
Parts:
- removed J2: Power in, My_Misc:BarrelJack_Horizontal
- removed X1: X322516MLB4SI, JLC2KiCad_Footprints:OSC-SMD_4P-L3.2-W2.5-BL
- added D1: LED, LED_SMD:LED_1206_3216Metric_Pad1.42x1.75mm_HandSolder, F.Cu at (161.3, 88.2)
- added J3: FTDI, Connector_PinHeader_2.54mm:PinHeader_1x06_P2.54mm_Vertical_SMD_Pin1Left, F.Cu at (133.0, 101.4)
- added J4: USB_C_Receptacle_PowerOnly_6P, Connector_USB:USB_C_Receptacle_GCT_USB4135-GF-A_6P_TopMnt_Horizontal, F.Cu at (144.1, 97.5)
- added JP1: FTDI Power, Button_Switch_SMD:SW_DIP_SPSTx01_Slide_6.7x4.1mm_W6.73mm_P2.54mm_LowProfile_JPin, F.Cu at (142.2, 116.6)
- added R2: 330R, Resistor_SMD:R_1206_3216Metric_Pad1.30x1.75mm_HandSolder, F.Cu at (132.0, 115.1)
- added R3: 5k1, Resistor_SMD:R_1206_3216Metric_Pad1.30x1.75mm_HandSolder, F.Cu at (132.0, 118.3)
- added R4: 5k1, Resistor_SMD:R_1206_3216Metric_Pad1.30x1.75mm_HandSolder, F.Cu at (132.0, 121.6)
- added Y1: 16MHz, Crystal:Crystal_SMD_HC49-SD, F.Cu at (139.8, 89.6)
- C1: value VE-100M1ETR-0405 -> 22u; footprint JLC2KiCad_Footprints:CAP-SMD_BD4.0-L4.3-W4.3-RD -> Capacitor_SMD:CP_Elec_4x5.3
- C2: value VE-100M1ETR-0405 -> 22p; footprint JLC2KiCad_Footprints:CAP-SMD_BD4.0-L4.3-W4.3-RD -> Capacitor_SMD:C_1206_3216Metric_Pad1.33x1.80mm_HandSolder
- C3: value 1206CG220J102NT -> 22p; footprint JLC2KiCad_Footprints:C1206 -> Capacitor_SMD:C_1206_3216Metric_Pad1.33x1.80mm_HandSolder
- C4: value 1206CG220J102NT -> 100n; footprint JLC2KiCad_Footprints:C1206 -> Capacitor_SMD:C_1206_3216Metric_Pad1.33x1.80mm_HandSolder
- C5: value CL31B104KBCNNNC -> 10u; footprint JLC2KiCad_Footprints:C1206 -> Capacitor_SMD:CP_Elec_5x5.4
- J1: value FTDI -> 2x3_ISP_header; footprint My_Headers:6-pin FTDI Programmer PinSocket large -> Connector_PinHeader_2.54mm:PinHeader_2x03_P2.54mm_Vertical_SMD
- R1: value 1206W4F1002T5E -> 10k; footprint JLC2KiCad_Footprints:R1206 -> Resistor_SMD:R_1206_3216Metric_Pad1.30x1.75mm_HandSolder
- U1: footprint JLC2KiCad_Footprints:SOT-223_L6.5-W3.5-P2.30-LS7.0-BR -> Package_TO_SOT_SMD:SOT-223
- U2: footprint JLC2KiCad_Footprints:TQFP-32_L7.0-W7.0-P0.80-LS9.0-BL -> Package_QFP:TQFP-32_7x7mm_P0.8mm
- moved U1 65.2 mm to (153.6, 116.0), turned to 0 degrees
- moved C2 63.3 mm to (161.5, 113.4)
- moved R1 60.7 mm to (132.0, 111.8)
- moved U2 56.9 mm to (142.8, 107.8)
- moved C4 44.4 mm to (161.5, 120.1)
- moved C1 41.2 mm to (154.4, 89.4)
- moved J1 37.7 mm to (155.1, 106.9)
- moved C3 36.6 mm to (161.5, 116.8), turned to 0 degrees
- moved C5 28.5 mm to (155.6, 96.2)
Connections:
- net A4 renamed A4/SDA
- net A5 renamed A5/SCL
- C1 pad 1: VCC -> Net-(C1-Pad1)
- C2 pad 1: Net-(C2-Pad1) -> GND
- C2 pad 2: GND -> XTAL1
- C3 pad 2: XTAL1 -> XTAL2
- C4 pad 1: GND -> +5V
- C4 pad 2: XTAL2 -> Net-(J3-DTR)
- C5 pad 1: Net-(C5-Pad1) -> VCC
- C5 pad 2: +5V -> GND
- J1 pad 1: GND -> D12/MISO
- J1 pad 2: unconnected-(J1-Pad2) -> +5V
- J1 pad 3: +5V -> D13/SCK
- J1 pad 4: D0/Rx -> D11/MOSI
- J1 pad 5: D1/Tx -> Reset
- J1 pad 6: Net-(C5-Pad1) -> GND
- U1 pad 2: Net-(C2-Pad1) -> Net-(C1-Pad1)
- U1 pad 4: Net-(C2-Pad1) -> Net-(C1-Pad1)
- U2 pad 15: D11 -> D11/MOSI
- U2 pad 16: D12 -> D12/MISO
- U2 pad 17: D13 -> D13/SCK
- U2 pad 20: unconnected-(U2-Pad20) -> Aref
